File: CAN_MITM_V1_Kicad.sch (KiCad schematic (older format))
At the start: 33 parts, among them IC2 SN65HVD234, IC3 SN65HVD234, U1 STM32F105RBT6 CPU, X1 8MHz

Commit message: Fixing wrong footprint on C11
Parts:
- C11: footprint Capacitor_SMD:C_0805_2012Metric -> Capacitor_SMD:CP_Elec_10x10
Changed lines of the file:
@@
 F 0 "C11" H 8500 1500 50  0000 L CNN
 F 1 "470uF 25V" H 8200 1350 50  0000 L CNN
-F 2 "Capacitor_SMD:C_0805_2012Metric" H 8838 1250 50  0001 C CNN
+F 2 "Capacitor_SMD:CP_Elec_10x10" H 8838 1250 50  0001 C CNN
 F 3 "~" H 8800 1400 50  0001 C CNN
 	1    8800 1400

Commit message: Routed PCB and updated some of the schematic
Parts:
- C13, C14: footprint Capacitor_SMD:C_0805_2012Metric -> Capacitor_Tantalum_SMD:CP_EIA-3528-21_Kemet-B
- CONN3: footprint TE_1-776275-1 -> 1-776275-1:TE_1-776275-1
Connections:
- net labels added: CAN2L
- net labels removed: CANH, CANL
Changed lines of the file:
@@
 F 0 "C14" H 10368 2196 50  0000 L CNN
 F 1 "100uF 6.3V" H 10368 2105 50  0000 L CNN
-F 2 "Capacitor_SMD:C_0805_2012Metric" H 10288 2000 50  0001 C CNN
+F 2 "Capacitor_Tantalum_SMD:CP_EIA-3528-21_Kemet-B" H 10288 2000 50  0001 C CNN
 F 3 "~" H 10250 2150 50  0001 C CNN
 	1    10250 2150
@@
 $EndComp
 Text Label 10250 3650 0    50   ~ 0
-CANL
+CAN1L
 Text Label 10250 3450 0    50   ~ 0
-CANH
+CAN1H
 Text Label 9050 3700 0    50   ~ 0
 GND
@@
 GND
 Text Label 10250 5450 0    50   ~ 0
-CANL
+CAN2L
 Text Label 10250 5250 0    50   ~ 0
-CANH
+CAN2H
 Text Label 9050 5500 0    50   ~ 0
 GND
@@
 F 0 "C13" H 9718 2196 50  0000 L CNN
 F 1 "100uF 6.3V" H 9718 2105 50  0000 L CNN
-F 2 "Capacitor_SMD:C_0805_2012Metric" H 9638 2000 50  0001 C CNN
+F 2 "Capacitor_Tantalum_SMD:CP_EIA-3528-21_Kemet-B" H 9638 2000 50  0001 C CNN
 F 3 "~" H 9600 2150 50  0001 C CNN
 	1    9600 2150
@@
 F 0 "CONN3" H 3557 7567 50  0000 C CNN
 F 1 "1-776275-1" H 3557 7476 50  0000 C CNN
-F 2 "TE_1-776275-1" H 3450 7000 50  0001 L BNN
+F 2 "1-776275-1:TE_1-776275-1" H 3450 7000 50  0001 L BNN
 F 3 "TE Connectivity" H 3450 7000 50  0001 L BNN
 F 4 "B7" H 3450 7000 50  0001 L BNN "Field4"
@@
 CAN1L
 Text Label 4350 7400 2    50   ~ 0
-CAN2H
+CAN2L
+Text Label 6050 7300 0    50   ~ 0
+BOOT0
 $EndSCHEMATC
